Commit message: Add a sick_lms1xx laser

File: jackal/jackal_description/urdf/accessories.urdf.xacro (robot description, xacro)
@@ -1,4 +1,6 @@
 <?xml version="1.0"?>
 <robot xmlns:xacro="http://www.ros.org/wiki/xacro">
+  <xacro:arg name="robot_namespace1" default="jackal1"/>
+  <!-- topic="$(optenv JACKAL_LASER_TOPIC front/scan) -->
   <!--
     As you add to this URDF, please be aware that both the robot and
@@ -19,11 +21,13 @@
       <hokuyo_ust10_mount prefix="$(optenv JACKAL_LASER_MOUNT front)"
                           parent_link="$(optenv JACKAL_LASER_MOUNT front)_mount"
-                          topic="$(optenv JACKAL_LASER_TOPIC front/scan)" />
+                          topic="$(optenv JACKAL_LASER_TOPIC front/scan)"
+                          robot_namespace="front" />
     </xacro:if>
     <xacro:unless value="$(optenv JACKAL_LASER_HOKUYO 0)">
       <xacro:include filename="$(find jackal_description)/urdf/accessories/sick_lms1xx_mount.urdf.xacro" />
       <sick_lms1xx_mount prefix="$(optenv JACKAL_LASER_MOUNT front)"
-                         parent_link="$(optenv JACKAL_LASER_MOUNT front)_mount"
-                         topic="$(optenv JACKAL_LASER_TOPIC front/scan)"/>
+                        parent_link="$(optenv JACKAL_LASER_MOUNT front)_mount"
+                         topic="$(optenv JACKAL_LASER_TOPIC front/scan)"
+                         robot_namespace="$(arg robot_namespace)"/>
     </xacro:unless>
   </xacro:if>

File: jackal/jackal_description/urdf/accessories/hokuyo_ust10.urdf.xacro (robot description, xacro)
@@ -1,7 +1,7 @@
 <?xml version="1.0"?>
-<robot xmlns:xacro="http://ros.org/wiki/xacro">
+<robot xmlns:xacro="http://www.ros.org/wiki/xacro">
   <xacro:macro name="hokuyo_ust10_mount" params="prefix topic parent_link">
     <xacro:macro name="hokuyo_ust10" params="frame:=laser topic:=scan sample_size:=720 update_rate:=50
-               min_angle:=-2.35619 max_angle:=2.35619 min_range:=0.1 max_range:=30.0 robot_namespace:=/">
+               min_angle:=-2.35619 max_angle:=2.35619 min_range:=0.1 max_range:=30.0 robot_namespace:=/" >
       <link name="${frame}">
         <inertial>

File: jackal/jackal_description/urdf/accessories/sick_lms1xx_mount.urdf.xacro (robot description, xacro)
@@ -27,5 +27,5 @@
 <robot xmlns:xacro="http://www.ros.org/wiki/xacro">
   <xacro:include filename="$(find lms1xx)/urdf/sick_lms1xx.urdf.xacro" />
-  <xacro:macro name="sick_lms1xx_mount" params="prefix topic parent_link">
+  <xacro:macro name="sick_lms1xx_mount" params="prefix topic parent_link robot_namespace:=/ topic:=scan sample_size:=720 update_rate:=50 min_angle:=-2.35619 max_angle:=2.35619 min_range:=0.1 max_range:=30.0">
     <sick_lms1xx frame="${prefix}_laser" topic="${topic}" />
     <joint name="${prefix}_laser_mount_joint" type="fixed">
@@ -54,4 +54,37 @@
       <material>Gazebo/DarkGrey</material>
     </gazebo>
+    <gazebo reference="${prefix}_laser">
+      <turnGravityOff>true</turnGravityOff>
+      <sensor type="ray" name="${prefix}_laser">
+        <pose>0 0 0 0 0 0</pose>
+        <visualize>false</visualize>
+        <update_rate>${update_rate}</update_rate>
+        <ray>
+          <scan>
+            <horizontal>
+              <samples>${sample_size}</samples>
+              <resolution>1</resolution>
+              <min_angle>${min_angle}</min_angle>
+              <max_angle>${max_angle}</max_angle>
+            </horizontal>
+          </scan>
+          <range>
+            <min>${min_range}</min>
+            <max>${max_range}</max>
+            <resolution>0.01</resolution>
+          </range>
+          <noise>
+            <type>gaussian</type>
+            <mean>0.0</mean>
+            <stddev>0.001</stddev>
+          </noise>
+        </ray>
+        <plugin name="gazebo_ros_laser" filename="libgazebo_ros_laser.so">
+          <topicName>${topic}</topicName>
+          <frameName>${prefix}_laser</frameName>
+          <robotNamespace>${robot_namespace}</robotNamespace>
+        </plugin>
+      </sensor>
+    </gazebo>
   </xacro:macro>
 </robot>

File: jackal/jackal_description/urdf/jackal.urdf.xacro (robot description, xacro)
@@ -229,5 +229,7 @@
        of these into the final description is controlled by optenv variables, which
        default each one to off.-->
-  <xacro:include filename="$(find jackal_description)/urdf/accessories.urdf.xacro" />
+  <xacro:include filename="$(find jackal_description)/urdf/accessories.urdf.xacro">
+    <xacro:arg name="robot_namespace1" value="$(arg robot_namespace)"/>
+  </xacro:include>
   <!-- Optional custom includes. -->
   <xacro:include filename="$(optenv JACKAL_URDF_EXTRAS empty.urdf)" />
